File: OpenDropV4/Electronics/ModulAdapter_universal/PCB/ModulAdapter_universal.kicad_pcb (KiCad board)
At the start: 2 copper layers, 100 x 69.5 mm, 57 parts, among them J1 Mini_Dimm_244, J2 Conn_01x24_Female, J3 Conn_02x02_Top_Bottom, J4 Conn_02x02_Top_Bottom, J5 Conn_02x03_Odd_Even, M1 Motor_DC, M2 Motor_DC, Q1 Q_NMOS_GSD, Q2 AO3401A, Q3 Q_NMOS_GSD, Q4 AO3401A, Q5 Q_NMOS_GSD, Q6 AO3401A, U1 TC78H660FTG, U2 HV507, U4 HV507, U5 SAMD21G18B, Y1 32 765

Commit message: getting our OpenDropv4 ready for refactor - removing deprecated (<v4) files
Other:
- net class 4mil removed
- net class Big removed
- net class Default removed
- net class Power removed
